File: pcb/esp32stepper.kicad_pcb (KiCad board)
At the start: 4 copper layers, 40 x 40 mm, 84 parts, among them J1 IO, J3 Display 0.96" 128x96, J4 Qwiic_Vertical, J5 Stepper, J6 PWR, J7 JTAG, J8 FAN, J9 USB_C_Receptacle_USB2.0_14P, Q1 IRLML9301, Q2 IRLML9301, SW1 BOOT, SW2 RST, SW3 B1, SW4 B2, U1 LM555xMM, U2 TMC2208-LA, U3 BME280, U4 ESP32-S3-MINI-1, U5 TPS56339DDC, U6 CH224K, U7 MPU-6050

Commit message: update
Parts:
- removed the C23 at (86.6, 128.0)
- removed the U7 at (90.0, 130.0)
- added C25: 100nF 50V, Capacitor_SMD:C_0603_1608Metric, F.Cu at (86.1, 139.6)
- added C26: C_Polarized, Capacitor_SMD:CP_Elec_5x5.4, F.Cu at (100.3, 139.6)
- added JP3: PWM, Jumper:SolderJumper-3_P1.3mm_Bridged12_RoundedPad1.0x1.5mm, B.Cu at (95.5, 125.9)
- added R27: 10k, Resistor_SMD:R_0402_1005Metric, F.Cu at (88.5, 133.4)
- added REF**: OSHW-Certification-Mark-Stacked_8x7mm_SilkScreen, OSHW_Certification_Mark:OSHW-Certification-Mark-Stacked_8x7mm_SilkScreen, F.Cu at (274.2, 174.3)
- added U3: MPU-9250, Sensor_Motion:InvenSense_QFN-24_3x3mm_P0.4mm, B.Cu at (90.0, 130.0)
- added U4: AS5048B, Package_SO:TSSOP-14_4.4x5mm_P0.65mm, B.Cu at (90.0, 130.0)
- C1: renamed from C4; footprint Capacitor_SMD:C_0402_1005Metric_Pad0.74x0.62mm_HandSolder -> Capacitor_SMD:C_0402_1005Metric
- C10: renamed from C16; value 100µF 35V -> 10µF 50V; footprint Capacitor_SMD:C_Elec_6.3x7.7 -> Capacitor_SMD:C_1206_3216Metric
- C12: renamed from C11; footprint Capacitor_SMD:C_0402_1005Metric_Pad0.74x0.62mm_HandSolder -> Capacitor_SMD:C_0402_1005Metric
- C13: renamed from C22; footprint Capacitor_SMD:C_0402_1005Metric_Pad0.74x0.62mm_HandSolder -> Capacitor_SMD:C_0402_1005Metric
- C15: renamed from C12; footprint Capacitor_SMD:C_0603_1608Metric_Pad1.08x0.95mm_HandSolder -> Capacitor_SMD:C_0603_1608Metric
- C16: renamed from C21; footprint Capacitor_SMD:C_0402_1005Metric_Pad0.74x0.62mm_HandSolder -> Capacitor_SMD:C_0402_1005Metric
- C17: renamed from C18; footprint Capacitor_SMD:C_0603_1608Metric_Pad1.08x0.95mm_HandSolder -> Capacitor_SMD:C_0603_1608Metric
- C19, C2: footprint Capacitor_SMD:C_0402_1005Metric_Pad0.74x0.62mm_HandSolder -> Capacitor_SMD:C_0402_1005Metric
- C20: renamed from C13; footprint Capacitor_SMD:C_0402_1005Metric_Pad0.74x0.62mm_HandSolder -> Capacitor_SMD:C_0402_1005Metric
- C21: renamed from C15; footprint Capacitor_SMD:C_0402_1005Metric_Pad0.74x0.62mm_HandSolder -> Capacitor_SMD:C_0402_1005Metric
- C22: renamed from C14; footprint Capacitor_SMD:C_0402_1005Metric_Pad0.74x0.62mm_HandSolder -> Capacitor_SMD:C_0402_1005Metric
- C23: renamed from C17; footprint Capacitor_SMD:C_0402_1005Metric_Pad0.74x0.62mm_HandSolder -> Capacitor_SMD:C_0402_1005Metric
- C24: renamed from C20; footprint Capacitor_SMD:C_0402_1005Metric_Pad0.74x0.62mm_HandSolder -> Capacitor_SMD:C_0402_1005Metric
- C3: renamed from C6; footprint Capacitor_SMD:C_0603_1608Metric_Pad1.08x0.95mm_HandSolder -> Capacitor_SMD:C_0402_1005Metric
- C4: renamed from C3; footprint Capacitor_SMD:C_0603_1608Metric_Pad1.08x0.95mm_HandSolder -> Capacitor_SMD:C_0603_1608Metric
- C5: value 100nF 35V -> 100nF 50V; footprint Capacitor_SMD:C_0603_1608Metric_Pad1.08x0.95mm_HandSolder -> Capacitor_SMD:C_0603_1608Metric
- C6: renamed from C7; footprint Capacitor_SMD:C_0603_1608Metric_Pad1.08x0.95mm_HandSolder -> Capacitor_SMD:C_0603_1608Metric
- C7: renamed from C9; value 1µF 35V -> 10µF 50V; footprint Capacitor_SMD:C_0603_1608Metric_Pad1.08x0.95mm_HandSolder -> Capacitor_SMD:C_1206_3216Metric
- C8: renamed from C10; value 1µF 35V -> 100nF 50V; footprint Capacitor_SMD:C_0603_1608Metric_Pad1.08x0.95mm_HandSolder -> Capacitor_SMD:C_0603_1608Metric
- C9: renamed from C8; footprint Capacitor_SMD:C_0402_1005Metric_Pad0.74x0.62mm_HandSolder -> Capacitor_SMD:C_0402_1005Metric
- H2: footprint MountingHole:MountingHole_3.2mm_M3_Pad_Via -> MountingHole:MountingHole_3.2mm_M3
- H3: renamed from H1; footprint MountingHole:MountingHole_3.2mm_M3_Pad_Via -> MountingHole:MountingHole_3.5mm
- Q1: renamed from Q2; moved to B.Cu
- R1: renamed from R4; footprint Resistor_SMD:R_0402_1005Metric_Pad0.72x0.64mm_HandSolder -> Resistor_SMD:R_0402_1005Metric
- R10: renamed from R6; footprint Resistor_SMD:R_0402_1005Metric_Pad0.72x0.64mm_HandSolder -> Resistor_SMD:R_0402_1005Metric
- R11: renamed from R8; footprint Resistor_SMD:R_0402_1005Metric_Pad0.72x0.64mm_HandSolder -> Resistor_SMD:R_0402_1005Metric
- R12: renamed from R26; footprint Resistor_SMD:R_0402_1005Metric_Pad0.72x0.64mm_HandSolder -> Resistor_SMD:R_0402_1005Metric; moved to B.Cu
- R13: renamed from R15; footprint Resistor_SMD:R_0402_1005Metric_Pad0.72x0.64mm_HandSolder -> Resistor_SMD:R_0402_1005Metric
- R15: renamed from R24; value 1k -> 10k
- R17: renamed from R10; footprint Resistor_SMD:R_0402_1005Metric_Pad0.72x0.64mm_HandSolder -> Resistor_SMD:R_0402_1005Metric
- R18: renamed from R14; footprint Resistor_SMD:R_0402_1005Metric_Pad0.72x0.64mm_HandSolder -> Resistor_SMD:R_0402_1005Metric
- R19: renamed from R17; footprint Resistor_SMD:R_0402_1005Metric_Pad0.72x0.64mm_HandSolder -> Resistor_SMD:R_0402_1005Metric
- R2: renamed from R1; footprint Resistor_SMD:R_0402_1005Metric_Pad0.72x0.64mm_HandSolder -> Resistor_SMD:R_0402_1005Metric
- R20: renamed from R18; footprint Resistor_SMD:R_0402_1005Metric_Pad0.72x0.64mm_HandSolder -> Resistor_SMD:R_0402_1005Metric
- R21: renamed from R9; footprint Resistor_SMD:R_0402_1005Metric_Pad0.72x0.64mm_HandSolder -> Resistor_SMD:R_0402_1005Metric
- R22: renamed from R16; footprint Resistor_SMD:R_0402_1005Metric_Pad0.72x0.64mm_HandSolder -> Resistor_SMD:R_0402_1005Metric
- R23: renamed from R13; footprint Resistor_SMD:R_0402_1005Metric_Pad0.72x0.64mm_HandSolder -> Resistor_SMD:R_0402_1005Metric
- R24: renamed from R19; footprint Resistor_SMD:R_0402_1005Metric_Pad0.72x0.64mm_HandSolder -> Resistor_SMD:R_0402_1005Metric
- R25: renamed from R22; footprint Resistor_SMD:R_0402_1005Metric_Pad0.72x0.64mm_HandSolder -> Resistor_SMD:R_0402_1005Metric
- R26: renamed from R20; footprint Resistor_SMD:R_0402_1005Metric_Pad0.72x0.64mm_HandSolder -> Resistor_SMD:R_0402_1005Metric
- R3: renamed from R7; footprint Resistor_SMD:R_0402_1005Metric_Pad0.72x0.64mm_HandSolder -> Resistor_SMD:R_0402_1005Metric
- R4: renamed from R12; footprint Resistor_SMD:R_0402_1005Metric_Pad0.72x0.64mm_HandSolder -> Resistor_SMD:R_0402_1005Metric
- R5: renamed from R21; footprint Resistor_SMD:R_0402_1005Metric_Pad0.72x0.64mm_HandSolder -> Resistor_SMD:R_0402_1005Metric
- R6: renamed from R3; footprint Resistor_SMD:R_0805_2012Metric_Pad1.20x1.40mm_HandSolder -> Resistor_SMD:R_0805_2012Metric
- R7: renamed from R11; footprint Resistor_SMD:R_0805_2012Metric_Pad1.20x1.40mm_HandSolder -> Resistor_SMD:R_0805_2012Metric
- R8: renamed from R2; footprint Resistor_SMD:R_0402_1005Metric_Pad0.72x0.64mm_HandSolder -> Resistor_SMD:R_0402_1005Metric
- R9: renamed from R5; footprint Resistor_SMD:R_0402_1005Metric_Pad0.72x0.64mm_HandSolder -> Resistor_SMD:R_0402_1005Metric
- moved J7 34.4 mm to (73.4, 126.6), turned to -90 degrees
- moved J4 34.3 mm to (107.3, 128.8), turned to 90 degrees
- moved J8 34.3 mm to (72.7, 136.7), turned to -90 degrees
- moved R12 26.9 mm to (103.3, 124.1), turned to 180 degrees
- moved C22 25.3 mm to (74.8, 120.1), turned to 180 degrees
- moved C21 24.3 mm to (77.0, 120.1), turned to 0 degrees
- moved L1 24.0 mm to (75.9, 123.3), turned to 90 degrees
- moved Q1 24.0 mm to (103.3, 126.6), turned to -90 degrees
- moved C17 23.5 mm to (72.0, 124.1), turned to 180 degrees
- moved R22 23.4 mm to (72.0, 130.8), turned to 180 degrees
- moved C7 23.2 mm to (95.8, 139.6), turned to 90 degrees
- moved C15 22.7 mm to (72.0, 125.6), turned to 180 degrees
- moved LOGO1 22.3 mm to (103.3, 120.3)
- moved R23 22.2 mm to (80.3, 131.6), turned to -90 degrees
- moved C8 21.7 mm to (93.9, 139.6), turned to 90 degrees
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- renumbered C24 to C11, C1 to C14, C25 to C18, H3 to H1, J7 to J1, J5 to J2, J1 to J4, J4 to J5, J8 to J6, J6 to J7, J9 to J8, JP4 to JP1, JP3 to JP2, D1 to LED1, D2 to LED2, Q1 to Q2, R25 to R14, R23 to R16, SW2 to SW1, SW1 to SW3, SW3 to SW4, SW4 to SW5, U2 to U1, U4 to U2, U1 to U5, U5 to U6, U6 to U7, U3 to U8
Connections:
- J2 pad 1: Net-(J5-Pin_1) -> Net-(J2-Pin_1)
- J2 pad 2: Net-(J5-Pin_2) -> Net-(J2-Pin_2)
- J2 pad 3: Net-(J5-Pin_3) -> Net-(J2-Pin_3)
- J2 pad 4: Net-(J5-Pin_4) -> Net-(J2-Pin_4)
- LED1 pad 1: unconnected-(D1-DOUT-Pad1) -> Net-(LED1-DOUT)
- LED1 pad 3: LED1 -> RGB
- LED2 pad 3: LED2 -> Net-(LED1-DOUT)
- Q1 pad 1: /IO3 -> /IO2
- R12 pad 2: /IO3 -> /IO2
- R14 pad 2: /IO1 -> /IO3
- R15 pad 2: /IO3 -> /IO1
- R16 pad 1: /IO3 -> /IO1
- U1 pad 1: Net-(J5-Pin_2) -> Net-(J2-Pin_4)
- U1 pad 21: Net-(J5-Pin_4) -> Net-(J2-Pin_1)
- U1 pad 24: Net-(J5-Pin_3) -> Net-(J2-Pin_2)
- U1 pad 26: Net-(J5-Pin_1) -> Net-(J2-Pin_3)
- U2 pad 10: /PD_UART -> MPU_INT
- U2 pad 11: CFG2 -> INDEX
- U2 pad 12: DIR -> DIAG
- U2 pad 13: /TMC_EN -> BTN1
- U2 pad 14: STEP -> RGB
- U2 pad 15: INDEX -> CFG3
- U2 pad 16: DIAG -> CFG2
- U2 pad 17: /MS2 -> DIR
- U2 pad 18: /MS1 -> STEP
- U2 pad 19: unconnected-(U4-GPIO15/U0RTS/ADC2_CH4/XTAL_32K_P-Pad19) -> /IO1
- U2 pad 20: unconnected-(U4-GPIO16/U0CTS/ADC2_CH5/XTAL_32K_N-Pad20) -> /IO3
- U2 pad 21: BTN1 -> Net-(U2-GPIO17/U1TXD/ADC2_CH6)
- U2 pad 22: MPU_INT -> /PD_UART
- U2 pad 25: BTN2 -> /MS2
- U2 pad 26: /TACHO -> unconnected-(U2-GPIO26-Pad26)
- U2 pad 27: CFG3 -> /MS1
- U2 pad 30: CFG1 -> /TMC_EN
- U2 pad 34: SCL -> /TACHO
- U2 pad 41: SDA -> SCL
- U2 pad 44: LED2 -> SDA
- U2 pad 5: LED1 -> PWM
- U2 pad 6: /IO3 -> BTN2
- U2 pad 8: /IO1 -> CFG1
- U5 pad 4: /IO1 -> /IO3
- U5 pad 7: /IO3 -> /IO1
Routing:
- net Net-(D3-K): track 33.2 -> 5.44 mm, vias 1 -> 0
- net /IO1: track 19.9 -> 46.8 mm, vias 0 -> 2
- net CFG2: track 28.8 -> 5.43 mm, vias 2 -> 0
- net Net-(J5-Pin_4): track 22.4 -> 0.00 mm, vias 1 -> 0
- net Net-(J5-Pin_3): track 22.4 -> 0.00 mm, vias 1 -> 0
- net Net-(LED1-DOUT): track 0.00 -> 21.3 mm, vias 0 -> 2
- net BTN2: track 26.8 -> 46.0 mm
- net Net-(J5-Pin_1): track 17.5 -> 0.00 mm, vias 1 -> 0
- net Net-(J5-Pin_2): track 16.4 -> 0.00 mm, vias 1 -> 0
- net RGB: track 0.00 -> 15.7 mm, vias 0 -> 2
- net /TXD: track 30.6 -> 15.6 mm, vias 2 -> 0
- net PWM: track 0.00 -> 13.8 mm, vias 0 -> 1
- net /PG: track 6.00 -> 19.1 mm
- net /TMC_EN: track 22.6 -> 9.44 mm, vias 2 -> 0
- net /IO2: track 25.9 -> 38.5 mm, vias 2 -> 3
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- added copper zone on B.Cu, net +3V3
- added copper zone on F.Cu, net Net-(J2-Pin_1)
- added copper zone on F.Cu, net Net-(J2-Pin_2)
- added copper zone on F.Cu, net Net-(J2-Pin_3)
- added copper zone on F.Cu, net Net-(J2-Pin_4)
- added copper zone on F.Cu, net Net-(U1-BRA)
- added copper zone on F.Cu, net Net-(U1-BRB)
- added copper zone on F.Cu, net VBUS
- added copper zone on B.Cu, net VDD
- removed copper zone on In2.Cu, net VBUS
Other:
- outline, holes or cut-outs redrawn
- board text added: "(bottom)"
- board text added: "0.017 mm"
- board text added: "0.02"
- board text added: "0.035 mm"
- board text added: "0.06 mm"
- board text added: "0.125 mm / 0.125 mm"
- board text added: "0.2 mm"
- board text added: "0.22 mm"
- board text added: "0.41 mm"
- board text added: "1.074 mm"
- board text added: "3.3"
- board text added: "4.5"
- board text added: "40 mm x 40 mm"
- board text added: "A"
- board text added: "B"
- board text added: "Black"
- board text added: "Boot Button"
- board text added: "Button1"
- board text added: "Button2"
- board text added: "Display Connector"
- board text added: "FR4 natural"
- board text added: "GPIO Connector"
- board text added: "QWIIC Connector"
- board text added: "RGB LED1"
- board text added: "RGB LED2"
- board text added: "Reset Button"
- board text added: "Stepper Connector"
- board text added: "USB-C Connector"
- board text added: "White"
- board text added: "alt. Power Connector"
- board text added: "max 24V!"
- board text removed: "0,017 mm"
- board text removed: "0,02"
- board text removed: "0,035 mm"
- board text removed: "0,06 mm"
- board text removed: "0,1250 mm / 0,1500 mm"
- board text removed: "0,2000 mm"
- board text removed: "0,22 mm"
- board text removed: "0,41 mm"
- board text removed: "1,0740 mm"
- board text removed: "3,3"
- board text removed: "4,5"
- board text removed: "40,0000 mm x 40,0000 mm"
- board text removed: "VDD"
