File: pcb/esp32stepper.kicad_pcb (KiCad board)
At the start: 4 copper layers, 40 x 40 mm, 84 parts, among them J1 IO, J3 Display 0.96" 128x96, J4 Qwiic_Vertical, J5 Stepper, J6 PWR, J7 JTAG, J8 FAN, J9 USB_C_Receptacle_USB2.0_14P, Q1 IRLML9301, Q2 IRLML9301, SW1 BOOT, SW2 RST, SW3 B1, SW4 B2, U1 LM555xMM, U2 TMC2208-LA, U3 BME280, U4 ESP32-S3-MINI-1, U5 TPS56339DDC, U6 CH224K, U7 MPU-6050

Commit message: add OSHW id
Parts:
- removed REF**: OSHW-Symbol_6.7x6mm_SilkScreen, Symbol:OSHW-Symbol_6.7x6mm_SilkScreen
- added LOGO1: ~, OSHW_Certification_Mark:OSHW-Certification-Mark-Stacked_8x7mm_SilkScreen, B.Cu at (91.2, 139.0)
Routing:
- net GND: vias 122 -> 123

Commit message: update
Parts:
- removed the C23 at (86.6, 128.0)
- removed the U7 at (90.0, 130.0)
- added JP3: PWM, Jumper:SolderJumper-3_P1.3mm_Bridged12_RoundedPad1.0x1.5mm, B.Cu at (84.9, 126.3)
- added REF**: OSHW-Certification-Mark-Stacked_8x7mm_SilkScreen, OSHW_Certification_Mark:OSHW-Certification-Mark-Stacked_8x7mm_SilkScreen, F.Cu at (274.2, 174.3)
- added U3: MPU-9250, Sensor_Motion:InvenSense_QFN-24_3x3mm_P0.4mm, B.Cu at (90.0, 130.0)
- added U4: AS5048B, Package_SO:TSSOP-14_4.4x5mm_P0.65mm, B.Cu at (90.0, 130.0)
- R15: renamed from R24; value 1k -> 10k
- moved D1 20.0 mm to (100.0, 113.5), turned to 90 degrees
- moved D2 20.0 mm to (80.0, 113.5)
- moved C16 8.20 mm to (89.8, 125.6), turned to 180 degrees
- moved C11 5.32 mm to (86.7, 128.8), turned to 90 degrees
- moved LOGO1 2.77 mm to (90.4, 136.3)
- moved C13 0.41 mm to (86.7, 131.0)
- renumbered C4 to C1, C16 to C10, C24 to C11, C11 to C12, C22 to C13, C1 to C14, C12 to C15, C21 to C16, C18 to C17, C25 to C18, C13 to C20, C15 to C21, C14 to C22, C17 to C23, C20 to C24, C6 to C3, C3 to C4, C7 to C6, C9 to C7, C10 to C8, C8 to C9, H3 to H1, H1 to H3, J7 to J1, J5 to J2, J1 to J4, J4 to J5, J8 to J6, J6 to J7, J9 to J8, JP4 to JP1, JP3 to JP2, Q2 to Q1, Q1 to Q2, R4 to R1, R6 to R10, R8 to R11, R26 to R12, R15 to R13, R25 to R14, R23 to R16, R10 to R17, R14 to R18, R17 to R19, R1 to R2, R18 to R20, R9 to R21, R16 to R22, R13 to R23, R19 to R24, R22 to R25, R20 to R26, R7 to R3, R12 to R4, R21 to R5, R3 to R6, R11 to R7, R2 to R8, R5 to R9, SW2 to SW1, SW1 to SW3, SW3 to SW4, SW4 to SW5, U2 to U1, U4 to U2, U1 to U5, U5 to U6, U6 to U7, U3 to U8
Connections:
- D1 pad 1: unconnected-(D1-DOUT-Pad1) -> Net-(D1-DOUT)
- D1 pad 3: LED1 -> RGB
- D2 pad 3: LED2 -> Net-(D1-DOUT)
- J4 pad 5: /IO3 -> /IO1
- J4 pad 7: /IO1 -> /IO3
- Q1 pad 1: /IO3 -> /IO2
- R12 pad 2: /IO3 -> /IO2
- R14 pad 2: /IO1 -> /IO3
- R15 pad 2: /IO3 -> /IO1
- R16 pad 1: /IO3 -> /IO1
- U2 pad 44: LED2 -> RGB
- U2 pad 5: LED1 -> /IO1
- U2 pad 6: /IO3 -> /IO2
- U2 pad 7: /IO2 -> /IO3
- U2 pad 8: /IO1 -> PWM
- U5 pad 4: /IO1 -> /IO3
- U5 pad 7: /IO3 -> /IO1
Routing:
- net Net-(D1-DOUT): track 0.00 -> 21.7 mm, vias 0 -> 2
- net Net-(JP3-C): track 0.00 -> 10.4 mm
- net LED2: track 10.3 -> 0.00 mm
- net RGB: track 0.00 -> 9.48 mm
- net LED1: track 8.81 -> 0.00 mm, vias 2 -> 0
- net SCL: track 30.0 -> 37.4 mm
- net /IO1: track 19.9 -> 26.1 mm
- net PWM: track 0.00 -> 5.74 mm, vias 0 -> 1
- net SDA: track 41.0 -> 37.3 mm
- net /IO2: track 25.9 -> 29.5 mm
- net Net-(U7-CPOUT): track 3.38 -> 0.00 mm
- net /TXD: track 30.6 -> 27.3 mm
- net /IO3: track 23.7 -> 20.7 mm
- net /RXD: track 28.6 -> 26.5 mm
- net MPU_INT: track 4.70 -> 3.07 mm
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- added copper zone on B.Cu, net +3V3
Other:
- outline, holes or cut-outs redrawn
- board text added: "A"
- board text added: "B"
- board text added: "Black"
- board text added: "Boot Button"
- board text added: "Button1"
- board text added: "Button2"
- board text added: "Display Connector"
- board text added: "FR4 natural"
- board text added: "GPIO Connector"
- board text added: "QWIIC Connector"
- board text added: "RGB LED1"
- board text added: "RGB LED2"
- board text added: "Reset Button"
- board text added: "Stepper Connector"
- board text added: "USB-C Connector (top)"
- board text added: "White"
- board text added: "external Power Connector (bottom)"

Commit message: major update to v1.1
Parts:
- added C25: 100nF 50V, Capacitor_SMD:C_0603_1608Metric, F.Cu at (86.1, 139.6)
- added R27: 10k, Resistor_SMD:R_0402_1005Metric, F.Cu at (88.2, 133.4)
- C1, C12, C13, C16, C19, C2, C20, C21, C22, C23, C24, C9: footprint Capacitor_SMD:C_0402_1005Metric_Pad0.74x0.62mm_HandSolder -> Capacitor_SMD:C_0402_1005Metric
- C10: value 100µF 35V -> 10µF 50V; footprint Capacitor_SMD:C_Elec_6.3x7.7 -> Capacitor_SMD:C_1206_3216Metric
- C15, C17, C4, C6: footprint Capacitor_SMD:C_0603_1608Metric_Pad1.08x0.95mm_HandSolder -> Capacitor_SMD:C_0603_1608Metric
- C3: footprint Capacitor_SMD:C_0603_1608Metric_Pad1.08x0.95mm_HandSolder -> Capacitor_SMD:C_0402_1005Metric
- C5: value 100nF 35V -> 100nF 50V; footprint Capacitor_SMD:C_0603_1608Metric_Pad1.08x0.95mm_HandSolder -> Capacitor_SMD:C_0603_1608Metric
- C7: value 1µF 35V -> 10µF 50V; footprint Capacitor_SMD:C_0603_1608Metric_Pad1.08x0.95mm_HandSolder -> Capacitor_SMD:C_1206_3216Metric
- C8: value 1µF 35V -> 100nF 50V; footprint Capacitor_SMD:C_0603_1608Metric_Pad1.08x0.95mm_HandSolder -> Capacitor_SMD:C_0603_1608Metric
- H2: footprint MountingHole:MountingHole_3.2mm_M3_Pad_Via -> MountingHole:MountingHole_3.2mm_M3
- H3: footprint MountingHole:MountingHole_3.2mm_M3_Pad_Via -> MountingHole:MountingHole_3.5mm
- Q1: moved to B.Cu
- R1, R10, R11, R13, R17, R18, R19, R2, R20, R21, R22, R23, R24, R25, R26, R3, R4, R5, R8, R9: footprint Resistor_SMD:R_0402_1005Metric_Pad0.72x0.64mm_HandSolder -> Resistor_SMD:R_0402_1005Metric
- R12: footprint Resistor_SMD:R_0402_1005Metric_Pad0.72x0.64mm_HandSolder -> Resistor_SMD:R_0402_1005Metric; moved to B.Cu
- R6, R7: footprint Resistor_SMD:R_0805_2012Metric_Pad1.20x1.40mm_HandSolder -> Resistor_SMD:R_0805_2012Metric
- moved J7 34.4 mm to (73.4, 126.6), turned to -90 degrees
- moved J4 34.3 mm to (107.3, 128.8), turned to 90 degrees
- moved J8 34.3 mm to (72.7, 136.7), turned to -90 degrees
- moved R12 26.9 mm to (103.3, 124.1), turned to 180 degrees
- moved C22 25.3 mm to (74.8, 120.1), turned to 180 degrees
- moved C21 24.3 mm to (77.0, 120.1), turned to 0 degrees
- moved L1 24.0 mm to (75.9, 123.3), turned to 90 degrees
- moved Q1 24.0 mm to (103.3, 126.6), turned to -90 degrees
- moved C17 23.5 mm to (72.0, 124.1), turned to 180 degrees
- moved R22 23.4 mm to (72.0, 130.8), turned to 180 degrees
- moved C7 23.2 mm to (95.8, 139.6), turned to 90 degrees
- moved C15 22.7 mm to (72.0, 125.6), turned to 180 degrees
- moved R23 22.2 mm to (80.3, 131.6), turned to -90 degrees
- moved C8 21.7 mm to (93.9, 139.6), turned to 90 degrees
- moved Q2 21.2 mm to (72.0, 128.3), turned to 90 degrees
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- renumbered D1 to LED1, D2 to LED2
Connections:
- J4 pad 5: /IO1 -> /IO3
- J4 pad 7: /IO3 -> /IO1
- U1 pad 1: Net-(J2-Pin_2) -> Net-(J2-Pin_4)
- U1 pad 21: Net-(J2-Pin_4) -> Net-(J2-Pin_1)
- U1 pad 24: Net-(J2-Pin_3) -> Net-(J2-Pin_2)
- U1 pad 26: Net-(J2-Pin_1) -> Net-(J2-Pin_3)
- U2 pad 10: /PD_UART -> MPU_INT
- U2 pad 11: CFG2 -> INDEX
- U2 pad 12: DIR -> DIAG
- U2 pad 14: STEP -> RGB
- U2 pad 15: INDEX -> CFG3
- U2 pad 16: DIAG -> CFG2
- U2 pad 18: /MS1 -> CFG1
- U2 pad 19: unconnected-(U2-GPIO15/U0RTS/ADC2_CH4/XTAL_32K_P-Pad19) -> /IO1
- U2 pad 20: unconnected-(U2-GPIO16/U0CTS/ADC2_CH5/XTAL_32K_N-Pad20) -> /IO3
- U2 pad 21: BTN1 -> Net-(U2-GPIO17/U1TXD/ADC2_CH6)
- U2 pad 22: MPU_INT -> /PD_UART
- U2 pad 25: BTN2 -> /MS1
- U2 pad 26: /TACHO -> unconnected-(U2-GPIO26-Pad26)
- U2 pad 27: CFG3 -> BTN1
- U2 pad 30: CFG1 -> BTN2
- U2 pad 34: SCL -> /TACHO
- U2 pad 41: SDA -> SCL
- U2 pad 44: RGB -> SDA
- U2 pad 5: /IO1 -> PWM
- U2 pad 6: /IO2 -> STEP
- U2 pad 7: /IO3 -> /IO2
- U2 pad 8: PWM -> DIR
Routing:
- net Net-(D3-K): track 34.8 -> 5.44 mm, vias 1 -> 0
- net CFG2: track 29.6 -> 5.46 mm, vias 2 -> 0
- net /IO1: track 26.1 -> 48.8 mm, vias 0 -> 2
- net Net-(J2-Pin_4): track 22.4 -> 0.00 mm, vias 1 -> 0
- net Net-(J2-Pin_3): track 22.4 -> 0.00 mm, vias 1 -> 0
- net Net-(J2-Pin_1): track 17.5 -> 0.00 mm, vias 1 -> 0
- net Net-(J2-Pin_2): track 16.4 -> 0.00 mm, vias 1 -> 0
- net CFG3: track 18.0 -> 5.47 mm, vias 2 -> 0
- net /PG: track 6.00 -> 18.5 mm
- net BTN1: track 25.3 -> 37.0 mm
- net SDA: track 37.3 -> 48.7 mm, vias 3 -> 2
- net /TXD: track 27.3 -> 16.1 mm, vias 2 -> 0
- net /PD_UART: track 14.5 -> 4.19 mm, vias 2 -> 0
- net SCL: track 37.4 -> 47.5 mm, vias 2 -> 1
- net /IO2: track 29.5 -> 37.6 mm, vias 2 -> 3
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- added copper zone on F.Cu, net Net-(J2-Pin_1)
- added copper zone on F.Cu, net Net-(J2-Pin_2)
- added copper zone on F.Cu, net Net-(J2-Pin_3)
- added copper zone on F.Cu, net Net-(J2-Pin_4)
- added copper zone on F.Cu, net Net-(U1-BRA)
- added copper zone on F.Cu, net Net-(U1-BRB)
- added copper zone on F.Cu, net VBUS
- added copper zone on B.Cu, net VDD
- removed copper zone on In2.Cu, net VBUS
Other:
- outline, holes or cut-outs redrawn
- board text added: "(bottom)"
- board text added: "USB-C Connector"
- board text added: "alt. Power Connector"
- board text removed: "USB-C Connector (top)"
- board text removed: "VDD"
- board text removed: "external Power Connector (bottom)"

Commit message: update pcb
Parts:
- moved R3 16.2 mm to (96.4, 133.9), turned to 0 degrees
- moved JP3 12.3 mm to (95.5, 125.9)
- moved JP2 7.07 mm to (95.5, 133.8), turned to 90 degrees
- moved C9 1.94 mm to (85.0, 135.4), turned to 180 degrees
- moved JP1 1.76 mm to (95.5, 130.2), turned to -90 degrees
- moved C19 0.95 mm to (84.0, 134.4)
- moved R20 0.95 mm to (84.0, 133.4)
- moved C5 0.65 mm to (95.9, 135.8)
- moved R27 0.31 mm to (88.5, 133.4)
- moved U5 0.20 mm to (85.5, 123.8)
- moved R14 0.15 mm to (86.2, 134.4)
- moved R15 0.15 mm to (86.2, 133.4)
Connections:
- U2 pad 13: /TMC_EN -> BTN1
- U2 pad 17: /MS2 -> DIR
- U2 pad 18: CFG1 -> STEP
- U2 pad 25: /MS1 -> /MS2
- U2 pad 27: BTN1 -> /MS1
- U2 pad 30: BTN2 -> /TMC_EN
- U2 pad 6: STEP -> BTN2
- U2 pad 8: DIR -> CFG1
Routing:
- net BTN2: track 24.3 -> 46.0 mm, vias 0 -> 2
- net /TMC_EN: track 21.0 -> 9.44 mm, vias 2 -> 0
- net /MS2: track 20.7 -> 9.34 mm
- net PWM: track 3.80 -> 13.8 mm
- net BTN1: track 37.0 -> 27.4 mm, vias 0 -> 2
- net /TACHO: track 20.4 -> 11.2 mm
- net +3V3: track 15.4 -> 23.4 mm, vias 32 -> 30
- net DIR: track 18.2 -> 10.5 mm, vias 2 -> 0
- net SCL: track 47.5 -> 54.8 mm
- net Net-(JP3-C): track 11.9 -> 4.64 mm
- net STEP: track 18.7 -> 26.0 mm
- net CFG1: track 12.4 -> 18.4 mm, vias 0 -> 2
- net /MS1: track 12.0 -> 7.76 mm
- net USB-: track 26.2 -> 23.6 mm
- net USB+: track 25.9 -> 23.6 mm
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
Commit message: mend
Other:
- board text added: "max 24V!"
Changed lines of the file:
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@@
 		(title "ESP32STEPPER")
 		(date "2025-05-02")
-		(rev "1.1")
+		(rev "1.2")
 		(company "Stefan Herold")
 		(comment 1 "License: https://ohwr.org/cern_ohl_w_v2.txt (CERN-OHL-W)")
@@
 		)
 		(property "Value" "MS2"
-			(at 0 2 90)
+			(at 0 1.9 270)
 			(unlocked yes)
-			(layer "F.SilkS")
-			(hide yes)
+			(layer "B.SilkS")
 			(effects
 				(font
@@
 		)
 		(property "Value" "PWM"
-			(at -0.65 1.95 270)
+			(at 0 1.9 270)
 			(unlocked yes)
-			(layer "F.SilkS")
-			(hide yes)
+			(layer "B.SilkS")
 			(effects
 				(font
@@
 		)
 		(property "Value" "MS1"
-			(at 0 1.9 270)
+			(at 0 -1.9 270)
 			(unlocked yes)
-			(layer "F.SilkS")
-			(hide yes)
+			(layer "B.SilkS")
 			(effects
 				(font
@@
 		)
 	)
+	(gr_text "max 24V!"
+		(at 74.8 121.2 0)
+		(layer "B.SilkS")
+		(effects
+			(font
+				(size 1 1)
+				(thickness 0.2)
+				(bold yes)
+			)
+			(justify mirror)
+		)
+	)
 	(gr_text "GND"
 		(at 106.9 134.2 0)
@@
 	)
 	(gr_text "${TITLE}"
-		(at 80.5 126.7 90)
+		(at 82 126.65 90)
 		(layer "B.SilkS")
 		(effects
@@
 	)
 	(gr_text "v${REVISION}/${CURRENT_DATE}"
-		(at 82.1 126.6 90)
+		(at 84 126.55 90)
 		(layer "B.SilkS")
 		(effects
