File: pcb/esp32stepper.kicad_sch (KiCad schematic)
At the start: 84 parts, among them J1 IO, J3 Display 0.96" 128x96, J4 Qwiic_Vertical, J5 Stepper, J6 PWR, J7 JTAG, J8 FAN, J9 USB_C_Receptacle_USB2.0_14P, Q1 IRLML9301, Q2 IRLML9301, SW1 BOOT, SW2 RST, SW3 B1, SW4 B2, SW5 RotaryEncoder, U1 LM555xMM, U2 TMC2208-LA, U3 BME280, U4 ESP32-S3-MINI-1, U5 TPS56339DDC, U6 CH224K, U7 MPU-6050

Commit message: add OSHW id
Parts:
- added LOGO1: ~, OSHW_Certification_Mark:OSHW-Certification-Mark-Stacked_8x7mm_SilkScreen, symbol OSHW_Certification_Mark:OSHW_Certification_Mark_Stacked_Medium
Changed lines of the file:
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@@
 	)
 	(symbol
+		(lib_id "OSHW_Certification_Mark:OSHW_Certification_Mark_Stacked_Medium")
+		(at 393.7 259.08 0)
+		(unit 1)
+		(exclude_from_sim no)
+		(in_bom no)
+		(on_board yes)
+		(dnp no)
+		(fields_autoplaced yes)
+		(property "Reference" "LOGO1"
+			(at 393.7 259.08 0)
+			(effects
+				(font
+					(size 1.27 1.27)
+				)
+				(hide yes)
+			)
+		)
+		(property "Value" "~"
+			(at 393.7 259.08 0)
+			(effects
+				(font
+					(size 1.27 1.27)
+				)
+				(hide yes)
+			)
+		)
+		(property "Footprint" "OSHW_Certification_Mark:OSHW-Certification-Mark-Stacked_8x7mm_SilkScreen"
+			(at 393.7 259.08 0)
+			(effects
+				(font
+					(size 1.27 1.27)
+				)
+				(hide yes)
+			)
+		)
+		(property "Datasheet" ""
+			(at 393.7 259.08 0)
+			(effects
+				(font
+					(size 1.27 1.27)
+				)
+				(hide yes)
+			)
+		)
+		(property "Description" "OSHW Certification Mark, Stacked"
+			(at 393.7 259.08 0)
+			(effects
+				(font
+					(size 1.27 1.27)
+				)
+				(hide yes)
+			)
+		)
+		(instances
+			(project ""
+				(path "/018f2c15-69ca-452c-96bb-f69d28cc93bc"
+					(reference "LOGO1")
+					(unit 1)
+				)
+			)
+		)
+	)
+	(symbol
 		(lib_id "Device:R")
 		(at 361.95 158.75 0)
@@
 					(unit 1)
 				)
-			)
-		)
-	)
-	(symbol
-		(lib_id "Graphic:Logo_Open_Hardware_Small")
-		(at 398.78 261.62 0)
-		(unit 1)
-		(exclude_from_sim no)
-		(in_bom no)
-		(on_board no)
-		(dnp no)
-		(fields_autoplaced yes)
-		(property "Reference" "#SYM1"
-			(at 398.78 254.635 0)
-			(effects
-				(font
-					(size 1.27 1.27)
-				)
-				(hide yes)
-			)
-		)
-		(property "Value" "Logo_Open_Hardware_Small"
-			(at 398.78 267.335 0)
-			(effects
-				(font
-					(size 1.27 1.27)
-				)
-				(hide yes)
-			)
-		)
-		(property "Footprint" "Symbol:OSHW-Logo2_7.3x6mm_SilkScreen"
-			(at 398.78 261.62 0)
-			(effects
-				(font
-					(size 1.27 1.27)
-				)
-				(hide yes)
-			)
-		)
-		(property "Datasheet" "~"
-			(at 398.78 261.62 0)
-			(effects
-				(font
-					(size 1.27 1.27)
-				)
-				(hide yes)
-			)
-		)
-		(property "Description" "Open Hardware logo, small"
-			(at 398.78 261.62 0)
-			(effects
-				(font
-					(size 1.27 1.27)
-				)
-				(hide yes)
-			)
-		)
-		(instances
-			(project ""
-				(path "/018f2c15-69ca-452c-96bb-f69d28cc93bc"
-					(reference "#SYM1")
-					(unit 1)
-				)

Commit message: update
Parts:
- removed C16: 100µF 35V, Capacitor_SMD:C_Elec_6.3x7.7, symbol Device:C_Polarized
- removed C23: 2,2nF 50V, Capacitor_SMD:C_0603_1608Metric_Pad1.08x0.95mm_HandSolder, symbol Device:C
- removed U7: MPU-6050, Sensor_Motion:InvenSense_QFN-24_4x4mm_P0.5mm, symbol Sensor_Motion:MPU-6050
- added C10: 10µF 50V, Capacitor_SMD:C_1206_3216Metric, symbol Device:C
- added C25: 100nF 50V, Capacitor_SMD:C_0603_1608Metric, symbol Device:C
- added C26: C_Polarized, Capacitor_SMD:CP_Elec_5x5.4, symbol Device:C_Polarized
- added JP3: PWM, Jumper:SolderJumper-3_P1.3mm_Bridged12_RoundedPad1.0x1.5mm, symbol Jumper:SolderJumper_3_Bridged12
- added R27: 10k, Resistor_SMD:R_0402_1005Metric, symbol Device:R
- added U3: MPU-9250, Sensor_Motion:InvenSense_QFN-24_3x3mm_P0.4mm, symbol Sensor_Motion:MPU-9250
- added U4: AS5048B, Package_SO:TSSOP-14_4.4x5mm_P0.65mm, symbol Sensor_Magnetic:AS5048B
- C1: renamed from C4; footprint Capacitor_SMD:C_0402_1005Metric_Pad0.74x0.62mm_HandSolder -> Capacitor_SMD:C_0402_1005Metric
- C11: renamed from C24; now not fitted; now left out of the parts list
- C12: renamed from C11; footprint Capacitor_SMD:C_0402_1005Metric_Pad0.74x0.62mm_HandSolder -> Capacitor_SMD:C_0402_1005Metric
- C13: renamed from C22; footprint Capacitor_SMD:C_0402_1005Metric_Pad0.74x0.62mm_HandSolder -> Capacitor_SMD:C_0402_1005Metric; Variant MPU -> (none)
- C14: renamed from C1; LCSC (none) -> C7432762
- C15: renamed from C12; footprint Capacitor_SMD:C_0603_1608Metric_Pad1.08x0.95mm_HandSolder -> Capacitor_SMD:C_0603_1608Metric
- C16: renamed from C21; footprint Capacitor_SMD:C_0402_1005Metric_Pad0.74x0.62mm_HandSolder -> Capacitor_SMD:C_0402_1005Metric; Variant MPU -> (none)
- C17: renamed from C18; footprint Capacitor_SMD:C_0603_1608Metric_Pad1.08x0.95mm_HandSolder -> Capacitor_SMD:C_0603_1608Metric
- C19, C2: footprint Capacitor_SMD:C_0402_1005Metric_Pad0.74x0.62mm_HandSolder -> Capacitor_SMD:C_0402_1005Metric
- C20: renamed from C13; footprint Capacitor_SMD:C_0402_1005Metric_Pad0.74x0.62mm_HandSolder -> Capacitor_SMD:C_0402_1005Metric
- C21: renamed from C15; footprint Capacitor_SMD:C_0402_1005Metric_Pad0.74x0.62mm_HandSolder -> Capacitor_SMD:C_0402_1005Metric
- C22: renamed from C14; footprint Capacitor_SMD:C_0402_1005Metric_Pad0.74x0.62mm_HandSolder -> Capacitor_SMD:C_0402_1005Metric
- C23: renamed from C17; footprint Capacitor_SMD:C_0402_1005Metric_Pad0.74x0.62mm_HandSolder -> Capacitor_SMD:C_0402_1005Metric
- C24: renamed from C20; footprint Capacitor_SMD:C_0402_1005Metric_Pad0.74x0.62mm_HandSolder -> Capacitor_SMD:C_0402_1005Metric
- C3: renamed from C6; footprint Capacitor_SMD:C_0603_1608Metric_Pad1.08x0.95mm_HandSolder -> Capacitor_SMD:C_0402_1005Metric; LCSC C915842 -> C380305
- C4: renamed from C3; footprint Capacitor_SMD:C_0603_1608Metric_Pad1.08x0.95mm_HandSolder -> Capacitor_SMD:C_0603_1608Metric
- C5: value 100nF 35V -> 100nF 50V; footprint Capacitor_SMD:C_0603_1608Metric_Pad1.08x0.95mm_HandSolder -> Capacitor_SMD:C_0603_1608Metric; LCSC C5342943 -> C91183
- C6: renamed from C7; footprint Capacitor_SMD:C_0603_1608Metric_Pad1.08x0.95mm_HandSolder -> Capacitor_SMD:C_0603_1608Metric
- C7: renamed from C9; value 1µF 35V -> 10µF 50V; footprint Capacitor_SMD:C_0603_1608Metric_Pad1.08x0.95mm_HandSolder -> Capacitor_SMD:C_1206_3216Metric; LCSC C7432774 -> C7432781
- C8: renamed from C10; value 1µF 35V -> 100nF 50V; footprint Capacitor_SMD:C_0603_1608Metric_Pad1.08x0.95mm_HandSolder -> Capacitor_SMD:C_0603_1608Metric; LCSC C7432774 -> C91183
- C9: renamed from C8; footprint Capacitor_SMD:C_0402_1005Metric_Pad0.74x0.62mm_HandSolder -> Capacitor_SMD:C_0402_1005Metric
- D3: now not fitted
- H2: symbol Mechanical:MountingHole_Pad -> Mechanical:MountingHole
- H3: renamed from H1; symbol Mechanical:MountingHole_Pad -> Mechanical:MountingHole
- J6: renamed from J8; now not fitted
- Q1: renamed from Q2; now not fitted
- R1: renamed from R4; footprint Resistor_SMD:R_0402_1005Metric_Pad0.72x0.64mm_HandSolder -> Resistor_SMD:R_0402_1005Metric
- R10: renamed from R6; footprint Resistor_SMD:R_0402_1005Metric_Pad0.72x0.64mm_HandSolder -> Resistor_SMD:R_0402_1005Metric; LCSC C304153 -> C854480
- R11: renamed from R8; footprint Resistor_SMD:R_0402_1005Metric_Pad0.72x0.64mm_HandSolder -> Resistor_SMD:R_0402_1005Metric; LCSC C304153 -> C854480
- R12: renamed from R26; footprint Resistor_SMD:R_0402_1005Metric_Pad0.72x0.64mm_HandSolder -> Resistor_SMD:R_0402_1005Metric; now not fitted
- R13: renamed from R15; footprint Resistor_SMD:R_0402_1005Metric_Pad0.72x0.64mm_HandSolder -> Resistor_SMD:R_0402_1005Metric; LCSC C304153 -> C854480
- R14: renamed from R25; LCSC (none) -> C304153
- R15: renamed from R24; value 1k -> 10k; LCSC (none) -> C304153
- R16: renamed from R23; LCSC (none) -> C93942
- R17: renamed from R10; footprint Resistor_SMD:R_0402_1005Metric_Pad0.72x0.64mm_HandSolder -> Resistor_SMD:R_0402_1005Metric; LCSC C304153 -> C854480
- R18: renamed from R14; footprint Resistor_SMD:R_0402_1005Metric_Pad0.72x0.64mm_HandSolder -> Resistor_SMD:R_0402_1005Metric
- R19: renamed from R17; footprint Resistor_SMD:R_0402_1005Metric_Pad0.72x0.64mm_HandSolder -> Resistor_SMD:R_0402_1005Metric; LCSC C304153 -> C854480
- R2: renamed from R1; footprint Resistor_SMD:R_0402_1005Metric_Pad0.72x0.64mm_HandSolder -> Resistor_SMD:R_0402_1005Metric
- R20: renamed from R18; footprint Resistor_SMD:R_0402_1005Metric_Pad0.72x0.64mm_HandSolder -> Resistor_SMD:R_0402_1005Metric; LCSC C2077651 -> C11702
- R21: renamed from R9; footprint Resistor_SMD:R_0402_1005Metric_Pad0.72x0.64mm_HandSolder -> Resistor_SMD:R_0402_1005Metric; LCSC C427218 -> C138003
- R22: renamed from R16; footprint Resistor_SMD:R_0402_1005Metric_Pad0.72x0.64mm_HandSolder -> Resistor_SMD:R_0402_1005Metric; LCSC C304153 -> C854480
- R23: renamed from R13; footprint Resistor_SMD:R_0402_1005Metric_Pad0.72x0.64mm_HandSolder -> Resistor_SMD:R_0402_1005Metric; LCSC C304153 -> C854480
- R24: renamed from R19; footprint Resistor_SMD:R_0402_1005Metric_Pad0.72x0.64mm_HandSolder -> Resistor_SMD:R_0402_1005Metric
- R25: renamed from R22; footprint Resistor_SMD:R_0402_1005Metric_Pad0.72x0.64mm_HandSolder -> Resistor_SMD:R_0402_1005Metric
- R26: renamed from R20; footprint Resistor_SMD:R_0402_1005Metric_Pad0.72x0.64mm_HandSolder -> Resistor_SMD:R_0402_1005Metric; LCSC C304153 -> C854480
- R3: renamed from R7; footprint Resistor_SMD:R_0402_1005Metric_Pad0.72x0.64mm_HandSolder -> Resistor_SMD:R_0402_1005Metric; LCSC C304153 -> C854480
- R4: renamed from R12; footprint Resistor_SMD:R_0402_1005Metric_Pad0.72x0.64mm_HandSolder -> Resistor_SMD:R_0402_1005Metric
- R5: renamed from R21; footprint Resistor_SMD:R_0402_1005Metric_Pad0.72x0.64mm_HandSolder -> Resistor_SMD:R_0402_1005Metric
- R6: renamed from R3; footprint Resistor_SMD:R_0805_2012Metric_Pad1.20x1.40mm_HandSolder -> Resistor_SMD:R_0805_2012Metric; LCSC C723643 -> C2935234
- R7: renamed from R11; footprint Resistor_SMD:R_0805_2012Metric_Pad1.20x1.40mm_HandSolder -> Resistor_SMD:R_0805_2012Metric; LCSC C723643 -> C2935234
- R8: renamed from R2; footprint Resistor_SMD:R_0402_1005Metric_Pad0.72x0.64mm_HandSolder -> Resistor_SMD:R_0402_1005Metric
- R9: renamed from R5; footprint Resistor_SMD:R_0402_1005Metric_Pad0.72x0.64mm_HandSolder -> Resistor_SMD:R_0402_1005Metric
- SW1: renamed from SW2; LCSC C221703 -> C221699
- SW3: renamed from SW1; LCSC C221703 -> C221699
- SW4: renamed from SW3; LCSC C221703 -> C221699
- SW5: renamed from SW4; LCSC C221703 -> C221699
- renumbered C25 to C18, H3 to H1, J7 to J1, J5 to J2, J1 to J4, J4 to J5, J6 to J7, J9 to J8, JP4 to JP1, JP3 to JP2, D1 to LED1, D2 to LED2, Q1 to Q2, SW5 to SW2, U2 to U1, U4 to U2, U1 to U5, U5 to U6, U6 to U7, U3 to U8
Connections:
- net +3V3: now also U3.1 (RESV_VDDIO), U3.13 (VDD), U3.22 (~{CS}), U3.8 (VDDIO), U4.11 (VDD5V), U4.12 (VDD3V)
- net BTN1: now also U2.13 (GPIO9/TOUCH9/ADC1_CH8/FSPIHD/SUBSPIHD); no longer U2.21 (GPIO17/U1TXD/ADC2_CH6)
- net BTN2: now also U2.6 (GPIO2/TOUCH2/ADC1_CH1); no longer U2.25 (GPIO21)
- net CFG1: now also U2.8 (GPIO4/TOUCH4/ADC1_CH3); no longer U2.30 (GPIO48/SPICLK_N/SUBSPICLK_N_DIFF)
- net CFG2: now also U2.16 (GPIO12/TOUCH12/ADC2_CH1/FSPICLK/FSPIIO6/SUBSPICLK); no longer U2.11 (GPIO7/TOUCH7/ADC1_CH6)
- net CFG3: now also U2.15 (GPIO11/TOUCH11/ADC2_CH0/FSPID/FSPIIO5/SUBSPID); no longer U2.27 (GPIO47/SPICLK_P/SUBSPICLK_P_DIFF)
- net DIAG: now also U2.12 (GPIO8/TOUCH8/ADC1_CH7/SUBSPICS1); no longer U2.16 (GPIO12/TOUCH12/ADC2_CH1/FSPICLK/FSPIIO6/SUBSPICLK)
- net DIR: now also U2.17 (GPIO13/TOUCH13/ADC2_CH2/FSPIQ/FSPIIO7/SUBSPIQ); no longer U2.12 (GPIO8/TOUCH8/ADC1_CH7/SUBSPICS1)
- net GND: now also C10.2, C25.2, C26.2, U3.11 (FSYNC), U3.18 (GND), U3.20 (RESV_GND), U3.9 (AD0/MISO), U4.10 (TEST), U4.13 (GND), U4.3 (A2), U4.4 (A1), U4.5 (TEST), U4.6 (TEST), U4.7 (TEST), U4.8 (TEST), U4.9 (TEST); no longer H2.1, H3.1
- net INDEX: now also U2.11 (GPIO7/TOUCH7/ADC1_CH6); no longer U2.15 (GPIO11/TOUCH11/ADC2_CH0/FSPID/FSPIIO5/SUBSPID)
- net IO1: now also R15.2, R16.1, U2.19 (GPIO15/U0RTS/ADC2_CH4/XTAL_32K_P), U5.7 (DIS); no longer R14.2, U2.8 (GPIO4/TOUCH4/ADC1_CH3), U5.4 (R)
- net IO2: now also Q1.1 (G), R12.2
- net IO3: now also R14.2, U2.20 (GPIO16/U0CTS/ADC2_CH5/XTAL_32K_N), U5.4 (R); no longer Q1.1 (G), R12.2, R15.2, R16.1, U2.6 (GPIO2/TOUCH2/ADC1_CH1), U5.7 (DIS)
- net MPU_INT: now also U2.10 (GPIO6/TOUCH6/ADC1_CH5), U3.12 (INT); no longer U2.22 (GPIO18/U1RXD/ADC2_CH7/CLK_OUT3)
- net MS1: now also U2.27 (GPIO47/SPICLK_P/SUBSPICLK_P_DIFF); no longer U2.18 (GPIO14/TOUCH14/ADC2_CH3/FSPIWP/FSPIDQS/SUBSPIWP)
- net MS2: now also U2.25 (GPIO21); no longer U2.17 (GPIO13/TOUCH13/ADC2_CH2/FSPIQ/FSPIIO7/SUBSPIQ)
- net SCL: now also U2.41 (GPIO45), U3.23 (SCL/SCLK), U4.2 (SCL); no longer U2.34 (GPIO38/FSPIWP/SUBSPIWP)
- net SDA: now also U2.44 (GPIO46), U3.24 (SDA/MOSI), U4.1 (SDA); no longer U2.41 (GPIO45)
- net STEP: now also U2.18 (GPIO14/TOUCH14/ADC2_CH3/FSPIWP/FSPIDQS/SUBSPIWP), JP3.3 (B); no longer U2.14 (GPIO10/TOUCH10/ADC1_CH9/FSPICS0/FSPIIO4/SUBSPICS0)
- net TACHO: now also U2.34 (GPIO38/FSPIWP/SUBSPIWP); no longer U2.26 (GPIO26)
- net VDD: now also C10.1, C25.1, C26.1
- net /PD_UART: now also U2.22 (GPIO18/U1RXD/ADC2_CH7/CLK_OUT3), R27.2; no longer U2.10 (GPIO6/TOUCH6/ADC1_CH5)
- net /TMC_EN: now also U2.30 (GPIO48/SPICLK_N/SUBSPICLK_N_DIFF); no longer U2.13 (GPIO9/TOUCH9/ADC1_CH8/FSPIHD/SUBSPIHD)
- net at LED1.1 (DOUT): now also LED2.3 (DIN)
- net at J2.1 (Pin_1): now also U1.21 (OA2); no longer U1.26 (OB1)
- net at J2.2 (Pin_2): now also U1.24 (OA1); no longer U1.1 (OB2)
- net at J2.3 (Pin_3): now also U1.26 (OB1); no longer U1.24 (OA1)
- net at J2.4 (Pin_4): now also U1.1 (OB2); no longer U1.21 (OA2)
- net at C11.1: now also U3.10 (REGOUT)
- net LED1 renamed PWM
- net PWM: now also JP3.1 (A); no longer LED1.3 (DIN)
- removed net LED2: LED2.3 (DIN), U2.44 (GPIO46)
- new net: R27.1, U2.21 (GPIO17/U1TXD/ADC2_CH6)
- new net: JP3.2 (C), U4.14 (PWM)
- new net RGB: LED1.3 (DIN), U2.14 (GPIO10/TOUCH10/ADC1_CH9/FSPICS0/FSPIIO4/SUBSPICS0)
- no-connect marks 11 -> 9
Other:
- note added: "Rotation Sensor options"
- note added: "or use potentiometer with LM555"
- note removed: "Accelormeter"
- moved on the sheet: C13, C15, C16, C17, C20, C21, C22, C24, C7, C8, H1, J2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
