File: pcb/esp32stepper.kicad_sch (KiCad schematic)
At the start: 85 parts, among them J1 IO, J3 Display 0.96" 128x96, J4 Qwiic_Vertical, J5 Stepper, J6 PWR, J7 JTAG, J8 FAN, J9 USB_C_Receptacle_USB2.0_14P, Q1 IRLML9301, Q2 IRLML9301, SW1 BOOT, SW2 RST, SW3 B1, SW4 B2, SW5 RotaryEncoder, U1 LM555xMM, U2 TMC2208-LA, U3 BME280, U4 ESP32-S3-MINI-1, U5 TPS56339DDC, U6 CH224K, U7 MPU-6050

Commit message: update
Parts:
- removed C23: 2,2nF 50V, Capacitor_SMD:C_0603_1608Metric_Pad1.08x0.95mm_HandSolder, symbol Device:C
- removed U7: MPU-6050, Sensor_Motion:InvenSense_QFN-24_4x4mm_P0.5mm, symbol Sensor_Motion:MPU-6050
- added JP3: PWM, Jumper:SolderJumper-3_P1.3mm_Bridged12_RoundedPad1.0x1.5mm, symbol Jumper:SolderJumper_3_Bridged12
- added U3: MPU-9250, Sensor_Motion:InvenSense_QFN-24_3x3mm_P0.4mm, symbol Sensor_Motion:MPU-9250
- added U4: AS5048B, Package_SO:TSSOP-14_4.4x5mm_P0.65mm, symbol Sensor_Magnetic:AS5048B
- C11: renamed from C24; now not fitted; now left out of the parts list
- C13: renamed from C22; Variant MPU -> (none)
- C14: renamed from C1; LCSC (none) -> C7432762
- C16: renamed from C21; Variant MPU -> (none)
- D3: now not fitted
- J6: renamed from J8; now not fitted
- Q1: renamed from Q2; now not fitted
- R12: renamed from R26; now not fitted
- R14: renamed from R25; LCSC (none) -> C304153
- R15: renamed from R24; value 1k -> 10k; LCSC (none) -> C304153
- R16: renamed from R23; LCSC (none) -> C93942
- SW1: renamed from SW2; LCSC C221703 -> C221699
- SW3: renamed from SW1; LCSC C221703 -> C221699
- SW4: renamed from SW3; LCSC C221703 -> C221699
- SW5: renamed from SW4; LCSC C221703 -> C221699
- renumbered C4 to C1, C16 to C10, C11 to C12, C12 to C15, C18 to C17, C25 to C18, C13 to C20, C15 to C21, C14 to C22, C17 to C23, C20 to C24, C6 to C3, C3 to C4, C7 to C6, C9 to C7, C10 to C8, C8 to C9, H3 to H1, H1 to H3, J7 to J1, J5 to J2, J1 to J4, J4 to J5, J6 to J7, J9 to J8, JP4 to JP1, JP3 to JP2, Q1 to Q2, R4 to R1, R6 to R10, R8 to R11, R15 to R13, R10 to R17, R14 to R18, R17 to R19, R1 to R2, R18 to R20, R9 to R21, R16 to R22, R13 to R23, R19 to R24, R22 to R25, R20 to R26, R7 to R3, R12 to R4, R21 to R5, R3 to R6, R11 to R7, R2 to R8, R5 to R9, SW5 to SW2, U2 to U1, U4 to U2, U1 to U5, U5 to U6, U6 to U7, U3 to U8
Connections:
- net +3V3: now also U3.1 (RESV_VDDIO), U3.13 (VDD), U3.22 (~{CS}), U3.8 (VDDIO), U4.11 (VDD5V), U4.12 (VDD3V)
- net GND: now also U3.11 (FSYNC), U3.18 (GND), U3.20 (RESV_GND), U3.9 (AD0/MISO), U4.10 (TEST), U4.13 (GND), U4.3 (A2), U4.4 (A1), U4.5 (TEST), U4.6 (TEST), U4.7 (TEST), U4.8 (TEST), U4.9 (TEST)
- net IO1: now also J4.5 (Pin_5), R15.2, R16.1, SW2.B, U2.5 (GPIO1/TOUCH1/ADC1_CH0), U5.7 (DIS); no longer J4.7 (Pin_7), R14.2, SW2.A, U2.8 (GPIO4/TOUCH4/ADC1_CH3), U5.4 (R)
- net IO2: now also Q1.1 (G), R12.2, U2.6 (GPIO2/TOUCH2/ADC1_CH1); no longer U2.7 (GPIO3/TOUCH3/ADC1_CH2)
- net IO3: now also J4.7 (Pin_7), R14.2, SW2.A, U2.7 (GPIO3/TOUCH3/ADC1_CH2), U5.4 (R); no longer J4.5 (Pin_5), Q1.1 (G), R12.2, R15.2, R16.1, SW2.B, U2.6 (GPIO2/TOUCH2/ADC1_CH1), U5.7 (DIS)
- net MPU_INT: now also U3.12 (INT)
- net SCL: now also U3.23 (SCL/SCLK), U4.2 (SCL)
- net SDA: now also U3.24 (SDA/MOSI), U4.1 (SDA)
- net STEP: now also JP3.3 (B)
- net at D1.1 (DOUT): now also D2.3 (DIN)
- net at C11.1: now also U3.10 (REGOUT)
- net LED1 renamed RGB
- net RGB: now also U2.44 (GPIO46); no longer U2.5 (GPIO1/TOUCH1/ADC1_CH0)
- removed net LED2: D2.3 (DIN), U2.44 (GPIO46)
- new net: JP3.2 (C), U4.14 (PWM)
- new net PWM: JP3.1 (A), U2.8 (GPIO4/TOUCH4/ADC1_CH3)
- no-connect marks 11 -> 10
Other:
- note added: "Rotation Sensor options"
- note added: "use potentiometer with LM555"
- note removed: "Accelormeter"
- moved on the sheet: C10, C13, C15, C16, C17, C20, C21, C22, C24, C7, C8, D2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

Commit message: major update to v1.1
Parts:
- removed C10: 100µF 35V, Capacitor_SMD:C_Elec_6.3x7.7, symbol Device:C_Polarized
- added C10: 10µF 50V, Capacitor_SMD:C_1206_3216Metric, symbol Device:C
- added C25: 100nF 50V, Capacitor_SMD:C_0603_1608Metric, symbol Device:C
- added R27: 10k, Resistor_SMD:R_0402_1005Metric, symbol Device:R
- C1, C12, C13, C16, C19, C2, C20, C21, C22, C23, C24, C9: footprint Capacitor_SMD:C_0402_1005Metric_Pad0.74x0.62mm_HandSolder -> Capacitor_SMD:C_0402_1005Metric
- C15, C17, C4, C6: footprint Capacitor_SMD:C_0603_1608Metric_Pad1.08x0.95mm_HandSolder -> Capacitor_SMD:C_0603_1608Metric
- C3: footprint Capacitor_SMD:C_0603_1608Metric_Pad1.08x0.95mm_HandSolder -> Capacitor_SMD:C_0402_1005Metric; LCSC C915842 -> (none)
- C5: value 100nF 35V -> 100nF 50V; footprint Capacitor_SMD:C_0603_1608Metric_Pad1.08x0.95mm_HandSolder -> Capacitor_SMD:C_0603_1608Metric; LCSC C5342943 -> (none)
- C7: value 1µF 35V -> 10µF 50V; footprint Capacitor_SMD:C_0603_1608Metric_Pad1.08x0.95mm_HandSolder -> Capacitor_SMD:C_1206_3216Metric; LCSC C7432774 -> (none)
- C8: value 1µF 35V -> 100nF 50V; footprint Capacitor_SMD:C_0603_1608Metric_Pad1.08x0.95mm_HandSolder -> Capacitor_SMD:C_0603_1608Metric; LCSC C7432774 -> (none)
- H2, H3: symbol Mechanical:MountingHole_Pad -> Mechanical:MountingHole
- R1, R12, R18, R2, R20, R21, R24, R25, R4, R5, R8, R9: footprint Resistor_SMD:R_0402_1005Metric_Pad0.72x0.64mm_HandSolder -> Resistor_SMD:R_0402_1005Metric
- R10, R11, R13, R17, R19, R22, R23, R26, R3: footprint Resistor_SMD:R_0402_1005Metric_Pad0.72x0.64mm_HandSolder -> Resistor_SMD:R_0402_1005Metric; LCSC C304153 -> C2654005
- R6, R7: footprint Resistor_SMD:R_0805_2012Metric_Pad1.20x1.40mm_HandSolder -> Resistor_SMD:R_0805_2012Metric; LCSC C723643 -> C2935234
- U3: LCSC (none) -> C71459
- renumbered D1 to LED1, D2 to LED2
Connections:
- net BTN1: now also U2.27 (GPIO47/SPICLK_P/SUBSPICLK_P_DIFF); no longer U2.21 (GPIO17/U1TXD/ADC2_CH6)
- net BTN2: now also U2.30 (GPIO48/SPICLK_N/SUBSPICLK_N_DIFF); no longer U2.25 (GPIO21)
- net CFG1: now also U2.18 (GPIO14/TOUCH14/ADC2_CH3/FSPIWP/FSPIDQS/SUBSPIWP); no longer U2.30 (GPIO48/SPICLK_N/SUBSPICLK_N_DIFF)
- net CFG2: now also U2.16 (GPIO12/TOUCH12/ADC2_CH1/FSPICLK/FSPIIO6/SUBSPICLK); no longer U2.11 (GPIO7/TOUCH7/ADC1_CH6)
- net CFG3: now also U2.15 (GPIO11/TOUCH11/ADC2_CH0/FSPID/FSPIIO5/SUBSPID); no longer U2.27 (GPIO47/SPICLK_P/SUBSPICLK_P_DIFF)
- net DIAG: now also U2.12 (GPIO8/TOUCH8/ADC1_CH7/SUBSPICS1); no longer U2.16 (GPIO12/TOUCH12/ADC2_CH1/FSPICLK/FSPIIO6/SUBSPICLK)
- net DIR: now also U2.8 (GPIO4/TOUCH4/ADC1_CH3); no longer U2.12 (GPIO8/TOUCH8/ADC1_CH7/SUBSPICS1)
- net GND: now also C10.2, C25.2; no longer H2.1, H3.1
- net INDEX: now also U2.11 (GPIO7/TOUCH7/ADC1_CH6); no longer U2.15 (GPIO11/TOUCH11/ADC2_CH0/FSPID/FSPIIO5/SUBSPID)
- net IO1: now also J4.7 (Pin_7), SW2.A, U2.19 (GPIO15/U0RTS/ADC2_CH4/XTAL_32K_P); no longer J4.5 (Pin_5), SW2.B, U2.5 (GPIO1/TOUCH1/ADC1_CH0)
- net IO2: now also U2.7 (GPIO3/TOUCH3/ADC1_CH2); no longer U2.6 (GPIO2/TOUCH2/ADC1_CH1)
- net IO3: now also J4.5 (Pin_5), SW2.B, U2.20 (GPIO16/U0CTS/ADC2_CH5/XTAL_32K_N); no longer J4.7 (Pin_7), SW2.A, U2.7 (GPIO3/TOUCH3/ADC1_CH2)
- net MPU_INT: now also U2.10 (GPIO6/TOUCH6/ADC1_CH5); no longer U2.22 (GPIO18/U1RXD/ADC2_CH7/CLK_OUT3)
- net MS1: now also U2.25 (GPIO21); no longer U2.18 (GPIO14/TOUCH14/ADC2_CH3/FSPIWP/FSPIDQS/SUBSPIWP)
- net PWM: now also U2.5 (GPIO1/TOUCH1/ADC1_CH0); no longer U2.8 (GPIO4/TOUCH4/ADC1_CH3)
- net RGB: now also U2.14 (GPIO10/TOUCH10/ADC1_CH9/FSPICS0/FSPIIO4/SUBSPICS0); no longer U2.44 (GPIO46)
- net SCL: now also U2.41 (GPIO45); no longer U2.34 (GPIO38/FSPIWP/SUBSPIWP)
- net SDA: now also U2.44 (GPIO46); no longer U2.41 (GPIO45)
- net STEP: now also U2.6 (GPIO2/TOUCH2/ADC1_CH1); no longer U2.14 (GPIO10/TOUCH10/ADC1_CH9/FSPICS0/FSPIIO4/SUBSPICS0)
- net TACHO: now also U2.34 (GPIO38/FSPIWP/SUBSPIWP); no longer U2.26 (GPIO26)
- net VDD: now also C10.1, C25.1
- net /PD_UART: now also U2.22 (GPIO18/U1RXD/ADC2_CH7/CLK_OUT3), R27.2; no longer U2.10 (GPIO6/TOUCH6/ADC1_CH5)
- net at J2.1 (Pin_1): now also U1.21 (OA2); no longer U1.26 (OB1)
- net at J2.2 (Pin_2): now also U1.24 (OA1); no longer U1.1 (OB2)
- net at J2.3 (Pin_3): now also U1.26 (OB1); no longer U1.24 (OA1)
- net at J2.4 (Pin_4): now also U1.1 (OB2); no longer U1.21 (OA2)
- new net: R27.1, U2.21 (GPIO17/U1TXD/ADC2_CH6)
- no-connect marks 10 -> 9
Other:
- note added: "or use potentiometer with LM555"
- note removed: "use potentiometer with LM555"
- moved on the sheet: H1

Commit message: update pcb
Connections:
- net BTN1: now also U2.13 (GPIO9/TOUCH9/ADC1_CH8/FSPIHD/SUBSPIHD); no longer U2.27 (GPIO47/SPICLK_P/SUBSPICLK_P_DIFF)
- net BTN2: now also U2.6 (GPIO2/TOUCH2/ADC1_CH1); no longer U2.30 (GPIO48/SPICLK_N/SUBSPICLK_N_DIFF)
- net CFG1: now also U2.8 (GPIO4/TOUCH4/ADC1_CH3); no longer U2.18 (GPIO14/TOUCH14/ADC2_CH3/FSPIWP/FSPIDQS/SUBSPIWP)
- net DIR: now also U2.17 (GPIO13/TOUCH13/ADC2_CH2/FSPIQ/FSPIIO7/SUBSPIQ); no longer U2.8 (GPIO4/TOUCH4/ADC1_CH3)
- net MS1: now also U2.27 (GPIO47/SPICLK_P/SUBSPICLK_P_DIFF); no longer U2.25 (GPIO21)
- net MS2: now also U2.25 (GPIO21); no longer U2.17 (GPIO13/TOUCH13/ADC2_CH2/FSPIQ/FSPIIO7/SUBSPIQ)
- net STEP: now also U2.18 (GPIO14/TOUCH14/ADC2_CH3/FSPIWP/FSPIDQS/SUBSPIWP); no longer U2.6 (GPIO2/TOUCH2/ADC1_CH1)
- net /TMC_EN: now also U2.30 (GPIO48/SPICLK_N/SUBSPICLK_N_DIFF); no longer U2.13 (GPIO9/TOUCH9/ADC1_CH8/FSPIHD/SUBSPIHD)
Changed lines of the file:
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@@
 	(wire
 		(pts
-			(xy 165.1 106.68) (xy 182.88 106.68)
+			(xy 165.1 106.68) (xy 170.18 106.68)
 		)
 		(stroke
@@
 	(wire
 		(pts
-			(xy 165.1 116.84) (xy 182.88 116.84)
+			(xy 165.1 116.84) (xy 184.15 116.84)
 		)
 		(stroke
@@
 	(wire
 		(pts
-			(xy 170.18 127) (xy 165.1 127)
+			(xy 184.15 127) (xy 165.1 127)
 		)
 		(stroke
@@
 	)
 	(label "MS2"
-		(at 182.88 106.68 180)
+		(at 184.15 116.84 180)
 		(effects
 			(font
@@
 	)
 	(label "MS1"
-		(at 182.88 116.84 180)
+		(at 184.15 127 180)
 		(effects
 			(font
@@
 	(global_label "BTN2"
 		(shape input)
-		(at 170.18 129.54 0)
+		(at 170.18 78.74 0)
 		(fields_autoplaced yes)
 		(effects
@@
 		)
 		(property "Intersheetrefs" "${INTERSHEET_REFS}"
-			(at 177.9428 129.54 0)
+			(at 177.9428 78.74 0)
 			(effects
 				(font
@@
 	(global_label "BTN1"
 		(shape input)
-		(at 170.18 127 0)
+		(at 170.18 96.52 0)
 		(fields_autoplaced yes)
 		(effects
@@
 		)
 		(property "Intersheetrefs" "${INTERSHEET_REFS}"
-			(at 177.9428 127 0)
+			(at 177.9428 96.52 0)
 			(effects
 				(font
@@
 	(global_label "{slash}TMC_EN"
 		(shape input)
-		(at 170.18 96.52 0)
+		(at 170.18 129.54 0)
 		(fields_autoplaced yes)
 		(effects
@@
 		)
 		(property "Intersheetrefs" "${INTERSHEET_REFS}"
-			(at 181.6318 96.52 0)
+			(at 181.6318 129.54 0)
 			(effects
 				(font
@@
 	(global_label "DIR"
 		(shape input)
-		(at 170.18 83.82 0)
+		(at 170.18 106.68 0)
 		(fields_autoplaced yes)
 		(effects
@@
 		)
 		(property "Intersheetrefs" "${INTERSHEET_REFS}"
-			(at 176.31 83.82 0)
+			(at 176.31 106.68 0)
 			(effects
 				(font
@@
 	(global_label "CFG1"
 		(shape input)
-		(at 170.18 109.22 0)
+		(at 170.18 83.82 0)
 		(fields_autoplaced yes)
 		(effects
@@
 		)
 		(property "Intersheetrefs" "${INTERSHEET_REFS}"
-			(at 178.0033 109.22 0)
+			(at 178.0033 83.82 0)
 			(effects
 				(font
@@
 	(global_label "STEP"
 		(shape input)
-		(at 170.18 78.74 0)
+		(at 170.18 109.22 0)
 		(fields_autoplaced yes)
 		(effects
@@
 		)
 		(property "Intersheetrefs" "${INTERSHEET_REFS}"
-			(at 177.7613 78.74 0)
+			(at 177.7613 109.22 0)
 			(effects
 				(font
